File: CAD/premier_jet/premier_jet/premier_jet.kicad_pcb (KiCad board)
At the start: 0 parts

Commit message: Update pcb
Parts:
- added C1: 22nF 50V, Capacitor_SMD:C_0603_1608Metric, F.Cu at (80.8, 69.5)
- added C10: 2u2 6.3V, Capacitor_SMD:C_0402_1005Metric, F.Cu at (77.4, 65.0)
- added C11: 2u2 6.3V, Capacitor_SMD:C_0402_1005Metric, F.Cu at (77.4, 56.3)
- added C12: 100u LOW ESR, Capacitor_SMD:CP_Elec_6.3x5.4, F.Cu at (84.1, 38.8)
- added C13: 100n, Capacitor_SMD:C_0402_1005Metric, F.Cu at (77.4, 67.0)
- added C14: 100n, Capacitor_SMD:C_0402_1005Metric, F.Cu at (77.4, 35.7)
- added C15: 100n, Capacitor_SMD:C_0402_1005Metric, F.Cu at (77.4, 37.7)
- added C16: 100n, Capacitor_SMD:C_0402_1005Metric, F.Cu at (77.4, 68.9)
- added C17: 100nF 16V, Capacitor_SMD:C_0402_1005Metric, F.Cu at (77.4, 39.7)
- added C18: 22nF 50V, Capacitor_SMD:C_0603_1608Metric, F.Cu at (80.8, 44.2)
- added C19: 100n, Capacitor_SMD:C_0402_1005Metric, F.Cu at (77.4, 41.6)
- added C2: 100nF 16V, Capacitor_SMD:C_0402_1005Metric, F.Cu at (77.4, 61.1)
- added C20: 2u2 6.3V, Capacitor_SMD:C_0402_1005Metric, F.Cu at (77.4, 43.6)
- added C21: 100n, Capacitor_SMD:C_0402_1005Metric, F.Cu at (50.0, 55.6)
- added C22: 100u LOW ESR, Capacitor_SMD:CP_Elec_6.3x5.4, F.Cu at (84.1, 64.2)
- added C23: 100n, Capacitor_SMD:C_0402_1005Metric, F.Cu at (50.0, 57.6)
- added C24: 100n, Capacitor_SMD:C_0402_1005Metric, F.Cu at (50.0, 59.5)
- added C25: 100n, Capacitor_SMD:C_0402_1005Metric, F.Cu at (50.0, 61.5)
- added C26: 100n, Capacitor_SMD:C_0402_1005Metric, F.Cu at (50.0, 63.5)
- added C27: 100n, Capacitor_SMD:C_0402_1005Metric, F.Cu at (50.0, 65.4)
- added C28: 1u, Capacitor_SMD:C_0402_1005Metric, F.Cu at (50.0, 67.4)
- added C29: 100n, Capacitor_SMD:C_0402_1005Metric, F.Cu at (50.0, 69.4)
- added C3: 100u LOW ESR, Capacitor_SMD:CP_Elec_6.3x5.4, F.Cu at (84.1, 51.5)
- added C4: 100n, Capacitor_SMD:C_0402_1005Metric, F.Cu at (77.4, 48.4)
- added C5: 100n, Capacitor_SMD:C_0402_1005Metric, F.Cu at (77.4, 50.4)
- added C6: 100nF 16V, Capacitor_SMD:C_0402_1005Metric, F.Cu at (77.4, 52.3)
- added C7: 100n, Capacitor_SMD:C_0402_1005Metric, F.Cu at (77.4, 63.0)
- added C8: 22nF 50V, Capacitor_SMD:C_0603_1608Metric, F.Cu at (80.8, 56.8)
- added C9: 100n, Capacitor_SMD:C_0402_1005Metric, F.Cu at (77.4, 54.3)
- added FB1: 120Ohm_5000mA, Inductor_SMD:L_0805_2012Metric, F.Cu at (58.0, 62.8)
- added FB10: 120Ohm_5000mA, Inductor_SMD:L_0805_2012Metric, F.Cu at (67.1, 65.5)
- added FB11: 120Ohm_5000mA, Inductor_SMD:L_0805_2012Metric, F.Cu at (67.1, 68.3)
- added FB12: 120Ohm_5000mA, Inductor_SMD:L_0805_2012Metric, F.Cu at (67.1, 71.0)
- added FB2: 120Ohm_5000mA, Inductor_SMD:L_0805_2012Metric, F.Cu at (58.0, 65.5)
- added FB3: 120Ohm_5000mA, Inductor_SMD:L_0805_2012Metric, F.Cu at (58.0, 68.3)
- added FB4: 120Ohm_5000mA, Inductor_SMD:L_0805_2012Metric, F.Cu at (58.0, 71.0)
- added FB5: 120Ohm_5000mA, Inductor_SMD:L_0805_2012Metric, F.Cu at (62.5, 62.8)
- added FB6: 120Ohm_5000mA, Inductor_SMD:L_0805_2012Metric, F.Cu at (62.5, 65.5)
- added FB7: 120Ohm_5000mA, Inductor_SMD:L_0805_2012Metric, F.Cu at (62.5, 68.3)
- added FB8: 120Ohm_5000mA, Inductor_SMD:L_0805_2012Metric, F.Cu at (62.5, 71.0)
- added FB9: 120Ohm_5000mA, Inductor_SMD:L_0805_2012Metric, F.Cu at (67.1, 62.8)
- added H1: MountingHole_Pad, MountingHole:MountingHole_3.2mm_M3_Pad, F.Cu at (44.6, 38.7)
- added H2: MountingHole_Pad, MountingHole:MountingHole_3.2mm_M3_Pad, F.Cu at (44.6, 46.7)
- added H3: MountingHole_Pad, MountingHole:MountingHole_3.2mm_M3_Pad, F.Cu at (44.6, 54.6)
- added H4: MountingHole_Pad, MountingHole:MountingHole_3.2mm_M3_Pad, F.Cu at (44.6, 62.6)
- added J1: Conn_01x03, Connector_PinHeader_2.54mm:PinHeader_1x03_P2.54mm_Vertical, F.Cu at (71.7, 63.7)
- added J2: Conn_01x04, Connector_PinHeader_2.54mm:PinHeader_1x04_P2.54mm_Vertical, F.Cu at (58.0, 51.5)
- added J3: Conn_01x04, Connector_PinHeader_2.54mm:PinHeader_1x04_P2.54mm_Vertical, F.Cu at (62.6, 51.5)
- added J4: Conn_01x04, Connector_PinHeader_2.54mm:PinHeader_1x04_P2.54mm_Vertical, F.Cu at (67.2, 51.5)
- added J6: Conn_02x07_Counter_Clockwise, Connector_PinHeader_2.54mm:PinHeader_2x07_P2.54mm_Vertical, F.Cu at (50.9, 37.1)
- added R1: 1k, Resistor_SMD:R_0402_1005Metric, F.Cu at (70.9, 50.2)
- added R2: 1k, Resistor_SMD:R_0402_1005Metric, F.Cu at (70.9, 52.2)
- added R3: 1k, Resistor_SMD:R_0402_1005Metric, F.Cu at (70.9, 54.2)
- added U4: STM32G474RETx, Package_QFP:LQFP-64_10x10mm_P0.5mm, F.Cu at (62.9, 42.0)
Other:
- copper layers 0 -> 2
