File: CAD/premier_jet/premier_jet/premier_jet.kicad_pcb (KiCad board)
At the start: 2 copper layers, 54 parts, among them J1 Conn_01x03, J2 Conn_01x04, J3 Conn_01x04, J4 Conn_01x04, J6 Conn_02x07_Counter_Clockwise, U4 STM32G474RETx

Commit message: Long overdue update
Parts:
- removed FB1, FB10, FB11, FB12, FB2, FB3, FB4, FB5, FB6, FB7, FB8, FB9: 120Ohm_5000mA, Inductor_SMD:L_0805_2012Metric
- added C30: 470p 100V, Capacitor_SMD:C_0603_1608Metric, F.Cu at (84.3, 148.0)
- added C31: 470u 100V, Capacitor_SMD:C_0603_1608Metric, F.Cu at (81.3, 148.0)
- added C32: 470u 100V, Capacitor_SMD:C_0603_1608Metric, F.Cu at (78.3, 148.0)
- added C33: 470u 100V, Capacitor_SMD:C_0603_1608Metric, F.Cu at (75.3, 148.0)
- added C34: 470u 100V, Capacitor_SMD:C_0603_1608Metric, F.Cu at (92.1, 148.0)
- added C35: 470u 100V, Capacitor_SMD:C_0603_1608Metric, F.Cu at (98.1, 148.0)
- added C36: 470u 100V, Capacitor_SMD:C_0603_1608Metric, F.Cu at (89.1, 148.0)
- added C37: 470u 100V, Capacitor_SMD:C_0603_1608Metric, F.Cu at (95.1, 148.0)
- added C38: 470u 100V, Capacitor_SMD:C_0603_1608Metric, F.Cu at (105.8, 148.0)
- added C39: 470u 100V, Capacitor_SMD:C_0603_1608Metric, F.Cu at (111.8, 148.0)
- added C40: 470u 100V, Capacitor_SMD:C_0603_1608Metric, F.Cu at (102.8, 148.0)
- added C41: 470u 100V, Capacitor_SMD:C_0603_1608Metric, F.Cu at (108.8, 148.0)
- added C42: 10u, Capacitor_SMD:C_0603_1608Metric, F.Cu at (66.5, 121.5)
- added G***: LOGO, veltest:veltest, F.Cu at (120.2, 140.5)
- added J5: Barrel_Jack_MountingPin, Connector_BarrelJack:BarrelJack_Wuerth_694106106102_2.0x5.5mm, F.Cu at (68.6, 106.5)
- added J7: USB_C_Receptacle_USB2.0_16P, Connector_USB:USB_C_Receptacle_GCT_USB4105-xx-A_16P_TopMnt_Horizontal, F.Cu at (121.2, 112.8)
- added R4: 5.1k, Resistor_SMD:R_0805_2012Metric, F.Cu at (114.5, 115.0)
- added R5: 5.1k, Resistor_SMD:R_0805_2012Metric, F.Cu at (114.5, 109.5)
- added U1: TMC2225-SA-T, TMC2225:HTSSOP28_TMC2225_TRI, F.Cu at (77.5, 130.0)
- added U2: TMC2225-SA-T, TMC2225:HTSSOP28_TMC2225_TRI, F.Cu at (95.0, 130.0)
- added U3: TMC2225-SA-T, TMC2225:HTSSOP28_TMC2225_TRI, F.Cu at (113.5, 130.0)
- added U5: BU33SD5WG-TR, BU33SD5WG:SSOP5_ROM, F.Cu at (82.5, 110.0)
- added U6: USBLC6-2SC6, Package_TO_SOT_SMD:SOT-23-6, F.Cu at (112.9, 112.2)
- J1: footprint Connector_PinHeader_2.54mm:PinHeader_1x03_P2.54mm_Vertical -> Connector_JST:JST_PH_B3B-PH-K_1x03_P2.00mm_Vertical
- J2, J3, J4: footprint Connector_PinHeader_2.54mm:PinHeader_1x04_P2.54mm_Vertical -> Connector_JST:JST_PH_B4B-PH-K_1x04_P2.00mm_Vertical
- J6: footprint Connector_PinHeader_2.54mm:PinHeader_2x07_P2.54mm_Vertical -> Connector_PinHeader_2.54mm:PinHeader_2x07_P2.54mm_Vertical_SMD
- moved H3 121.6 mm to (120.0, 150.0)
- moved H1 113.1 mm to (65.0, 150.0)
- moved J2 109.5 mm to (103.8, 151.0)
- moved C14 106.2 mm to (111.5, 136.3)
- moved C15 105.3 mm to (111.5, 137.3)
- moved C12 103.2 mm to (107.0, 139.5), turned to 180 degrees
- moved J3 103.2 mm to (90.0, 151.0)
- moved C17 101.5 mm to (111.5, 135.2)
- moved J4 99.9 mm to (76.2, 151.0)
- moved C18 95.0 mm to (108.8, 135.0), turned to 180 degrees
- moved C19 92.5 mm to (118.5, 124.5), turned to 180 degrees
- moved C20 91.6 mm to (118.5, 125.5)
- moved H2 89.6 mm to (120.0, 95.0)
- moved C4 89.5 mm to (93.0, 136.5)
- moved C5 88.5 mm to (93.0, 137.5)
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Connections:
- J2 pad 1: Net-(J2-Pin_1) -> /Motor2/OA1
- J2 pad 2: Net-(J2-Pin_2) -> /Motor2/OA2
- J2 pad 3: Net-(J2-Pin_3) -> /Motor2/OB1
- J2 pad 4: Net-(J2-Pin_4) -> /Motor2/OB2
- J3 pad 1: Net-(J3-Pin_1) -> /Motor1/OA1
- J3 pad 2: Net-(J3-Pin_2) -> /Motor1/OA2
- J3 pad 3: Net-(J3-Pin_3) -> /Motor1/OB1
- J3 pad 4: Net-(J3-Pin_4) -> /Motor1/OB2
- J4 pad 1: Net-(J4-Pin_1) -> /Motor/OA1
- J4 pad 2: Net-(J4-Pin_2) -> /Motor/OA2
- J4 pad 3: Net-(J4-Pin_3) -> /Motor/OB1
- J4 pad 4: Net-(J4-Pin_4) -> /Motor/OB2
- U4 pad 45: unconnected-(U4-PA11-Pad45) -> /USB_DN
- U4 pad 46: unconnected-(U4-PA12-Pad46) -> /USB_DP
Routing:
- net GND: track 0.00 -> 233.9 mm, vias 0 -> 106
- net /+5V: track 0.00 -> 110.2 mm, vias 0 -> 29
- net /+3.3V: track 0.00 -> 102.4 mm, vias 0 -> 7
- net /MS2: track 0.00 -> 55.1 mm, vias 0 -> 6
- net /MS1: track 0.00 -> 54.9 mm, vias 0 -> 2
- net /UART_RXTX_1: track 0.00 -> 43.0 mm, vias 0 -> 2
- net /DIR_3: track 0.00 -> 41.5 mm, vias 0 -> 2
- net /UART_RXTX_3: track 0.00 -> 36.1 mm, vias 0 -> 2
- net /PWM_NEOPIXEL: track 0.00 -> 35.8 mm, vias 0 -> 2
- net /CHOPPER_MODE_3: track 0.00 -> 33.7 mm, vias 0 -> 2
- net /PWM_MOTOR_3: track 0.00 -> 32.3 mm, vias 0 -> 2
- net /UART_RXTX_2: track 0.00 -> 30.6 mm, vias 0 -> 2
- net /T_VCP_TX: track 0.00 -> 30.1 mm, vias 0 -> 2
- net /PWM_MOTOR_1: track 0.00 -> 27.8 mm
- net /PWM_MOTOR_2: track 0.00 -> 27.5 mm, vias 0 -> 4
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- added copper zone on In2.Cu, net /+5V
- added copper zone on B.Cu, net GND
- added copper zone on F.Cu, net GND
- added copper zone on In1.Cu, net GND
Other:
- board outline added: 65 x 65 mm
- copper layers 2 -> 4
- board text added: "MANSARD Johann EyeOT Maker ENSEA 2A"
