File: CAD/premier_jet/premier_jet/motor.kicad_sch (KiCad schematic)
At the start: 10 parts, among them U1 TMC2225-SA-T

Commit message: Update pcb
Parts:
- C1: footprint (none) -> Capacitor_SMD:C_0603_1608Metric
- C10, C13, C16, C2, C7: footprint (none) -> Capacitor_SMD:C_0402_1005Metric
- C22: footprint (none) -> Capacitor_SMD:CP_Elec_6.3x5.4
- U1: footprint HTSSOP28_TMC2225_TRI -> (none)
Changed lines of the file:
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@@
 			)
 		)
-		(property "Footprint" ""
+		(property "Footprint" "Capacitor_SMD:CP_Elec_6.3x5.4"
 			(at 62.5348 93.98 0)
 			(effects
@@
 			)
 		)
-		(property "Footprint" ""
+		(property "Footprint" "Capacitor_SMD:C_0402_1005Metric"
 			(at 102.5652 91.44 0)
 			(effects
@@
 			)
 		)
-		(property "Footprint" ""
+		(property "Footprint" "Capacitor_SMD:C_0603_1608Metric"
 			(at 102.87 49.8348 0)
 			(effects
@@
 			)
 		)
-		(property "Footprint" ""
+		(property "Footprint" "Capacitor_SMD:C_0402_1005Metric"
 			(at 89.8652 101.6 0)
 			(effects
@@
 			)
 		)
-		(property "Footprint" ""
+		(property "Footprint" "Capacitor_SMD:C_0402_1005Metric"
 			(at 168.91 49.8348 0)
 			(effects
@@
 		(dnp no)
 		(property "Reference" "U1"
-			(at 130.556 42.164 0)
+			(at 128.016 82.55 0)
 			(effects
 				(font
@@
 		)
 		(property "Value" "TMC2225-SA-T"
-			(at 125.222 44.45 0)
+			(at 121.92 84.582 0)
 			(effects
 				(font
@@
 			)
 		)
-		(property "Footprint" "HTSSOP28_TMC2225_TRI"
+		(property "Footprint" ""
 			(at 107.95 50.8 0)
 			(effects
@@
 			)
 		)
-		(property "Footprint" ""
+		(property "Footprint" "Capacitor_SMD:C_0402_1005Metric"
 			(at 77.1652 101.6 0)
 			(effects
@@
 			)
 		)
-		(property "Footprint" ""
+		(property "Footprint" "Capacitor_SMD:C_0402_1005Metric"
 			(at 70.8152 101.6 0)
 			(effects
@@
 	)
 	(symbol
+		(lib_name "TMC2225-SA-T_1")
 		(lib_id "TMC2225-SA-T:TMC2225-SA-T")
 		(at 107.95 88.9 0)
@@
 			)
 		)
-		(property "Footprint" "HTSSOP28_TMC2225_TRI"
+		(property "Footprint" ""
 			(at 107.95 88.9 0)
 			(effects

Commit message: Long overdue update
Parts:
- removed SenseR1, SenseR2: R, symbol Device:R
- U1: footprint (none) -> TMC2225:HTSSOP28_TMC2225_TRI
Connections:
- net GND: now also U1.6 (BRA), U1.9 (BRB)
Changed lines of the file:
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@@
-	(wire
-		(pts
-			(xy 92.71 71.12) (xy 95.25 71.12)
-		)
-		(stroke
-			(width 0)
-			(type default)
-		)
-	)
 	(wire
 		(pts
@@
 	(wire
 		(pts
+			(xy 105.41 71.12) (xy 107.95 71.12)
+		)
+		(stroke
+			(width 0)
+			(type default)
+		)
+	)
+	(wire
+		(pts
 			(xy 107.95 99.06) (xy 104.14 99.06)
 		)
@@
 	(wire
 		(pts
-			(xy 102.87 74.93) (xy 105.41 74.93)
-		)
-		(stroke
-			(width 0)
-			(type default)
-		)
-	)
-	(wire
-		(pts
 			(xy 69.85 91.44) (xy 72.39 91.44)
 		)
@@
 	(wire
 		(pts
-			(xy 92.71 74.93) (xy 95.25 74.93)
-		)
-		(stroke
-			(width 0)
-			(type default)
-		)
-	)
-	(wire
-		(pts
 			(xy 101.6 91.44) (xy 107.95 91.44)
 		)
@@
 	(wire
 		(pts
+			(xy 104.14 114.3) (xy 107.95 114.3)
+		)
+		(stroke
+			(width 0)
+			(type default)
+		)
+	)
+	(wire
+		(pts
 			(xy 105.41 73.66) (xy 107.95 73.66)
 		)
@@
 	(wire
 		(pts
-			(xy 104.14 114.3) (xy 107.95 114.3)
-		)
-		(stroke
-			(width 0)
-			(type default)
-		)
-	)
-	(wire
-		(pts
-			(xy 105.41 74.93) (xy 105.41 73.66)
-		)
-		(stroke
-			(width 0)
-			(type default)
-		)
-	)
-	(wire
-		(pts
 			(xy 76.2 92.71) (xy 78.74 92.71)
-		)
-		(stroke
-			(width 0)
-			(type default)
-		)
-	)
-	(wire
-		(pts
-			(xy 102.87 71.12) (xy 107.95 71.12)
 		)
 		(stroke
@@
 	)
 	(symbol
-		(lib_id "Device:R")
-		(at 99.06 74.93 90)
-		(unit 1)
-		(exclude_from_sim no)
-		(in_bom yes)
-		(on_board yes)
-		(dnp no)
-		(property "Reference" "SenseR2"
-			(at 97.79 77.216 90)
-			(effects
-				(font
-					(size 1.27 1.27)
-				)
-			)
-		)
-		(property "Value" "R"
-			(at 99.06 78.994 90)
-			(effects
-				(font
-					(size 1.27 1.27)
-				)
-			)
-		)
-		(property "Footprint" ""
-			(at 99.06 76.708 90)
-			(effects
-				(font
-					(size 1.27 1.27)
-				)
-				(hide yes)
-			)
-		)
-		(property "Datasheet" "~"
-			(at 99.06 74.93 0)
-			(effects
-				(font
-					(size 1.27 1.27)
-				)
-				(hide yes)
-			)
-		)
-		(property "Description" "Resistor"
-			(at 99.06 74.93 0)
-			(effects
-				(font
-					(size 1.27 1.27)
-				)
-				(hide yes)
-			)
-		)
-		(pin "2"
-		)
-		(pin "1"
-		)
-		(instances
-			(project "premier_jet"
-				(path "/36d3f7e8-0ea0-47ce-aa05-c602f0df039a/038b460e-26c2-4ffb-a900-d66a9e1f3def"
-					(reference "SenseR6")
-					(unit 1)
-				)
-				(path "/36d3f7e8-0ea0-47ce-aa05-c602f0df039a/8788187e-ff99-4e1b-8eaf-42d1f137c9be"
-					(reference "SenseR4")
-					(unit 1)
-				)
-				(path "/36d3f7e8-0ea0-47ce-aa05-c602f0df039a/fbfd92f2-dab5-408f-a544-30223ba7d99a"
-					(reference "SenseR2")
-					(unit 1)
-				)
-			)
-		)
-	)
-	(symbol
 		(lib_id "power:GND")
 		(at 95.25 82.55 270)
@@
 	)
 	(symbol
-		(lib_id "Device:R")
-		(at 99.06 71.12 90)
-		(unit 1)
-		(exclude_from_sim no)
-		(in_bom yes)
-		(on_board yes)
-		(dnp no)
-		(property "Reference" "SenseR1"
-			(at 99.06 69.088 90)
-			(effects
-				(font
-					(size 1.27 1.27)
-				)
-			)
-		)
-		(property "Value" "R"
-			(at 99.06 73.152 90)
-			(effects
-				(font
-					(size 1.27 1.27)
-				)
-			)
-		)
-		(property "Footprint" ""
-			(at 99.06 72.898 90)
-			(effects
-				(font
-					(size 1.27 1.27)
-				)
-				(hide yes)
-			)
-		)
-		(property "Datasheet" "~"
-			(at 99.06 71.12 0)
-			(effects
-				(font
-					(size 1.27 1.27)
-				)
-				(hide yes)
-			)
-		)
-		(property "Description" "Resistor"
-			(at 99.06 71.12 0)
-			(effects
-				(font
-					(size 1.27 1.27)
-				)
-				(hide yes)
-			)
-		)
-		(pin "2"
-		)
-		(pin "1"
-		)
-		(instances
-			(project "premier_jet"
-				(path "/36d3f7e8-0ea0-47ce-aa05-c602f0df039a/038b460e-26c2-4ffb-a900-d66a9e1f3def"
-					(reference "SenseR5")
-					(unit 1)
-				)
-				(path "/36d3f7e8-0ea0-47ce-aa05-c602f0df039a/8788187e-ff99-4e1b-8eaf-42d1f137c9be"
-					(reference "SenseR3")
-					(unit 1)
-				)
-				(path "/36d3f7e8-0ea0-47ce-aa05-c602f0df039a/fbfd92f2-dab5-408f-a544-30223ba7d99a"
-					(reference "SenseR1")
-					(unit 1)
-				)
-			)
-		)
-	)
-	(symbol
 		(lib_id "power:GND")
 		(at 104.14 106.68 270)
@@
 			)
 		)
-		(property "Footprint" ""
+		(property "Footprint" "TMC2225:HTSSOP28_TMC2225_TRI"
 			(at 107.95 50.8 0)
 			(effects
@@
 	(symbol
 		(lib_id "power:GND")
-		(at 92.71 74.93 270)
+		(at 105.41 73.66 270)
 		(unit 1)
 		(exclude_from_sim no)
@@
 		(fields_autoplaced yes)
 		(property "Reference" "#PWR035"
-			(at 86.36 74.93 0)
+			(at 99.06 73.66 0)
 			(effects
 				(font
@@
 		)
 		(property "Value" "GND"
-			(at 88.9 74.9299 90)
+			(at 101.6 73.6599 90)
 			(effects
 				(font
@@
 		)
 		(property "Footprint" ""
-			(at 92.71 74.93 0)
+			(at 105.41 73.66 0)
 			(effects
 				(font
@@
 		)
 		(property "Datasheet" ""
-			(at 92.71 74.93 0)
+			(at 105.41 73.66 0)
 			(effects
 				(font
@@
 		)
 		(property "Description" "Power symbol creates a global label with name \"GND\" , ground"
-			(at 92.71 74.93 0)
+			(at 105.41 73.66 0)
 			(effects
 				(font
@@
 			)
 		)
-		(property "Footprint" ""
+		(property "Footprint" "TMC2225:HTSSOP28_TMC2225_TRI"
 			(at 107.95 88.9 0)
 			(effects
@@
 	(symbol
 		(lib_id "power:GND")
-		(at 92.71 71.12 270)
+		(at 105.41 71.12 270)
 		(unit 1)
 		(exclude_from_sim no)
@@
 		(fields_autoplaced yes)
 		(property "Reference" "#PWR038"
-			(at 86.36 71.12 0)
+			(at 99.06 71.12 0)
 			(effects
 				(font
@@
 		)
 		(property "Value" "GND"
-			(at 88.9 71.1199 90)
+			(at 101.6 71.1199 90)
 			(effects
 				(font
@@
 		)
 		(property "Footprint" ""
-			(at 92.71 71.12 0)
+			(at 105.41 71.12 0)
 			(effects
 				(font
@@
 		)
 		(property "Datasheet" ""
-			(at 92.71 71.12 0)
+			(at 105.41 71.12 0)
 			(effects
 				(font
@@
 		)
 		(property "Description" "Power symbol creates a global label with name \"GND\" , ground"
-			(at 92.71 71.12 0)
-			(effects
-				(font
+			(at 105.41 71.12 0)
+			(effects
+				(font
